File: Sterownik CPLD dla TFT LCD.kicad_pcb (KiCad board)
At the start: 2 copper layers, 140 x 92 mm, 183 parts, among them J1 Conn_01x02, J10 5V select, J11 IO_5V, J13 VGA, J14 RGB_LSB, J15 Audio Out, J2 Conn_01x02, J3 PDI, J4 JTAG, J5 Conn_01x40, J6 Micro_SD_Card, J7 9V AC, J8 9V AC, J9 5V DC, Q1 BSS138, Q2 BSS138, Q3 BSS138, Q4 BSS138, Q5 BSS138, Q6 BSS138, Q7 BSS138, Q8 BSS138, SW1 Reset, SW2 IO_3V3_ON/OFF, U1 XC2C256_VQ100, U10 74LS573, U11 74AHC1G00, U12 LM1117-1.8, U13 L7805, U14 RT9293, U15 MIC2289_MILF8, U16 PCF8563T, U17 ADV7123_TQFP48, U18 TPA2005, U19 74AHCT1GU04, U2 LM1117-3.3, U20 74AHCT1GU04, U3 ATxmega128A1-AU, U4 NAND_Flash_TSOP48, U5 SRAM_1024Kx16bit_TSOP48I, U6 74AHC1G00, U7 SRAM_1024Kx16bit_TSOP48I, U8 74LS573, U9 SRAM_512Kx16bit_TSOP44II, X1 IQXO-70, X2 IQXO-70, Y1 32768Hz

Commit message: I-sze zmiany
Parts:
- removed C47, C48, C49, C50, C51, C52, C53, C54, C7: 100nF, Capacitor_SMD:C_1206_3216Metric
- removed C55: 2n2, Capacitor_SMD:C_1206_3216Metric
- removed D2: 1N5819, Diode_SMD:D_SOD-123
- removed D3: 1N4148, Diode_SMD:D_MiniMELF
- removed F1: Fuse, Fuse:Fuse_1812_4532Metric
- removed J1, J2: Conn_01x02, Jumper:SolderJumper-2_P1.3mm_Open_RoundedPad1.0x1.5mm
- removed J10: 5V select, Connector_PinHeader_2.54mm:PinHeader_1x03_P2.54mm_Vertical
- removed J11: IO_5V, Connector_PinHeader_2.54mm:PinHeader_2x11_P2.54mm_Horizontal
- removed J8: 9V AC, Jacek:Zlacze_srubowe_2x_5mm
- removed L1: 10uH, Inductor_SMD:L_Taiyo-Yuden_NR-40xx
- removed L2: 22uH, Inductor_SMD:L_Taiyo-Yuden_NR-40xx
- removed Q3, Q4, Q5, Q6, Q7, Q8: BSS138, Package_TO_SOT_SMD:SOT-23
- removed R13: 2R2, Resistor_SMD:R_1206_3216Metric
- removed R14, R26, R27, R28, R29, R30, R31, R32, R33, R34, R35, R36, R37: 10k, Resistor_SMD:R_0603_1608Metric
- removed R15: 4k7, Resistor_SMD:R_1206_3216Metric
- removed R16: 7R5, Resistor_SMD:R_1206_3216Metric
- removed SW2: IO_3V3_ON/OFF, Button_Switch_THT:SW_DIP_SPSTx08_Slide_6.7x21.88mm_W7.62mm_P2.54mm_LowProfile
- removed U14: RT9293, Package_TO_SOT_SMD:TSOT-23-6
- removed U15: MIC2289_MILF8, Jacek:MLF8
- removed X2: IQXO-70, Oscillator:Oscillator_SMD_IQD_IQXO70-4Pin_7.5x5.0mm
- U16: footprint Package_SO:SOIC-8_3.9x4.9mm_P1.27mm -> Package_SO:SO-8_3.9x4.9mm_P1.27mm
- U17: moved to B.Cu
- moved C57 19.0 mm to (102.3, 135.2), turned to 270 degrees
- moved C56 16.9 mm to (102.9, 141.1)
- moved D5 16.9 mm to (105.9, 147.9)
- moved D4 16.9 mm to (108.2, 147.9)
- moved R21 16.9 mm to (110.6, 147.9)
- moved Y1 16.9 mm to (106.6, 144.0)
- moved JP11 16.9 mm to (113.1, 147.9)
- moved D6 16.9 mm to (103.5, 147.9)
- moved R17 16.9 mm to (101.1, 147.9)
- moved R23 14.5 mm to (191.6, 66.7)
- moved R25 14.1 mm to (193.3, 66.7)
- moved R18 12.4 mm to (105.7, 125.2), turned to 180 degrees
- moved U16 12.2 mm to (107.1, 133.8), turned to 180 degrees
- moved R20 11.7 mm to (105.7, 129.8), turned to 180 degrees
- moved R19 11.6 mm to (105.7, 127.5), turned to 180 degrees
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Connections:
- C6 pad 1: Net-(C6-Pad1) -> +3V3
- J13 pad 11: Net-(J13-Pad11) -> (no net)
- J13 pad 12: Net-(J13-Pad12) -> (no net)
- J13 pad 15: Net-(J13-Pad15) -> (no net)
- J13 pad 4: Net-(J13-Pad4) -> (no net)
- J13 pad 9: Net-(J13-Pad9) -> (no net)
- J3 pad 3: Net-(J3-Pad3) -> (no net)
- J3 pad 4: Net-(J3-Pad4) -> (no net)
- J4 pad 6: Net-(J4-Pad6) -> (no net)
- J4 pad 7: Net-(J4-Pad7) -> (no net)
- J4 pad 8: Net-(J4-Pad8) -> (no net)
- J5 pad 1: VLED- -> +5V
- J5 pad 2: VLED+ -> +5V
- J5 pad 23: B2 -> (no net)
- J5 pad 35: Net-(J5-Pad35) -> (no net)
- J5 pad 37: X+ -> (no net)
- J5 pad 38: Y+ -> (no net)
- J5 pad 39: X- -> (no net)
- J5 pad 40: Y- -> (no net)
- J5 pad 7: R2 -> (no net)
- J6 pad 12: Net-(J6-Pad12) -> (no net)
- J7 pad 3: Net-(J7-Pad3) -> (no net)
- J9 pad 1: 5V_DC -> +5V
- U1 pad 1: G6 -> G7
- U1 pad 10: PCLK -> HSYNC
- U1 pad 11: DISP -> VSYNC
- U1 pad 12: HSYNC -> DE
- U1 pad 13: VSYNC -> (no net)
- U1 pad 14: DE -> (no net)
- U1 pad 15: ATX1 -> ATX0
- U1 pad 16: ATX2 -> ATX1
- U1 pad 17: ATX3 -> ATX2
- U1 pad 18: ATX4 -> ATX3
- U1 pad 19: ATX5 -> ATX4
- U1 pad 2: G7 -> B3
- U1 pad 22: Ext_clk -> ATX5
- U1 pad 27: CLK_Out -> Ext_clk
- U1 pad 3: B2 -> B4
- U1 pad 4: B3 -> B5
- U1 pad 6: B4 -> B6
- U1 pad 7: B5 -> B7
- U1 pad 8: B6 -> PCLK
- U1 pad 87: R2 -> R3
- U1 pad 89: R3 -> R4
- U1 pad 9: B7 -> DISP
- U1 pad 90: R4 -> R5
- U1 pad 91: R5 -> R6
- U1 pad 92: R6 -> R7
- U1 pad 93: R7 -> G2
- U1 pad 94: G2 -> G3
- U1 pad 95: G3 -> G4
- U1 pad 96: G4 -> G5
- U1 pad 97: G5 -> G6
- U10 pad 12: Net-(U10-Pad12) -> (no net)
- U10 pad 13: Net-(U10-Pad13) -> (no net)
- U10 pad 14: Net-(U10-Pad14) -> (no net)
- U10 pad 15: Net-(U10-Pad15) -> (no net)
- U17 pad 18: B2 -> RGB_VCC_GND
- U17 pad 43: R2 -> RGB_VCC_GND
- U3 pad 1: X- -> ATX9
- U3 pad 10: ATX3 -> ATX2
- U3 pad 100: Y+ -> ATX10
- U3 pad 11: ATX2 -> ATX1
- U3 pad 12: ATX1 -> ATX0
- U3 pad 16: PWM_EN_LED -> (no net)
- U3 pad 2: Y- -> ATX8
- U3 pad 22: CLK_Out -> (no net)
- U3 pad 28: SD_CD -> (no net)
- U3 pad 29: SD_CS -> (no net)
- U3 pad 30: SD_CLK -> (no net)
- U3 pad 31: SD_MISO -> (no net)
- U3 pad 32: SD_MOSI -> (no net)
- U3 pad 35: IO1_ATX -> (no net)
- U3 pad 36: IO2_ATX -> (no net)
- U3 pad 37: IO3_ATX -> (no net)
- U3 pad 38: IO4_ATX -> SD_CD
- U3 pad 39: IO5_ATX -> SD_CS
- U3 pad 40: IO6_ATX -> SD_CLK
- U3 pad 41: IO7_ATX -> SD_MISO
- U3 pad 42: IO8_ATX -> SD_MOSI
- U3 pad 5: ATX8 -> ATX7
- U3 pad 6: ATX7 -> ATX6
- U3 pad 7: ATX6 -> ATX5
- U3 pad 8: ATX5 -> ATX4
- U3 pad 85: ATX15 -> (no net)
- U3 pad 86: ATX14 -> (no net)
- U3 pad 87: ATX13 -> (no net)
- U3 pad 88: ATX12 -> (no net)
- U3 pad 9: ATX4 -> ATX3
- U3 pad 91: X2_EN -> (no net)
- U3 pad 92: ATX_Clk -> (no net)
- U3 pad 95: ATX11 -> ATX15
- U3 pad 96: ATX10 -> ATX14
- U3 pad 97: ATX9 -> ATX13
- U3 pad 98: X1_EN -> ATX12
- U3 pad 99: X+ -> ATX11
- U4 pad 1: Net-(U4-Pad1) -> (no net)
- U4 pad 10: Net-(U4-Pad10) -> (no net)
- U4 pad 11: Net-(U4-Pad11) -> (no net)
- U4 pad 14: Net-(U4-Pad14) -> (no net)
- U4 pad 15: Net-(U4-Pad15) -> (no net)
- U4 pad 2: Net-(U4-Pad2) -> (no net)
- U4 pad 20: Net-(U4-Pad20) -> (no net)
- U4 pad 21: Net-(U4-Pad21) -> (no net)
- U4 pad 22: Net-(U4-Pad22) -> (no net)
- U4 pad 23: Net-(U4-Pad23) -> (no net)
- U4 pad 24: Net-(U4-Pad24) -> (no net)
- U4 pad 25: Net-(U4-Pad25) -> (no net)
- U4 pad 26: Net-(U4-Pad26) -> (no net)
- U4 pad 27: Net-(U4-Pad27) -> (no net)
- U4 pad 28: Net-(U4-Pad28) -> (no net)
- U4 pad 3: Net-(U4-Pad3) -> (no net)
- U4 pad 33: Net-(U4-Pad33) -> (no net)
- U4 pad 34: Net-(U4-Pad34) -> (no net)
- U4 pad 35: Net-(U4-Pad35) -> (no net)
- U4 pad 38: Net-(U4-Pad38) -> (no net)
- U4 pad 39: Net-(U4-Pad39) -> (no net)
- U4 pad 4: Net-(U4-Pad4) -> (no net)
- U4 pad 40: Net-(U4-Pad40) -> (no net)
- U4 pad 45: Net-(U4-Pad45) -> (no net)
- U4 pad 46: Net-(U4-Pad46) -> (no net)
- U4 pad 47: Net-(U4-Pad47) -> (no net)
- U4 pad 48: Net-(U4-Pad48) -> (no net)
- U4 pad 5: Net-(U4-Pad5) -> (no net)
- U4 pad 6: Net-(U4-Pad6) -> (no net)
- U5 pad 19: Net-(U5-Pad19) -> (no net)
- U5 pad 31: Net-(U5-Pad31) -> (no net)
- U5 pad 6: Net-(U5-Pad6) -> (no net)
- U7 pad 19: Net-(U7-Pad19) -> (no net)
- U7 pad 31: Net-(U7-Pad31) -> (no net)
- U7 pad 6: Net-(U7-Pad6) -> (no net)
- X1 pad 1: X1_EN -> (no net)
- X1 pad 4: Net-(C6-Pad1) -> +3V3
Routing:
- net GND: track 1340.7 -> 1020.6 mm, vias 183 -> 151
- net +5V: track 303.4 -> 173.2 mm, vias 26 -> 12
- net +3V3: track 875.0 -> 774.5 mm, vias 53 -> 43
- net PWM_EN_LED: track 84.5 -> 0.00 mm, vias 5 -> 0
- net R2: track 84.0 -> 0.00 mm, vias 1 -> 0
- net (no net): track 0.00 -> 74.2 mm, vias 0 -> 4
- net PCF_SCL: track 73.4 -> 5.57 mm, vias 3 -> 0
- net VLED-: track 67.0 -> 0.00 mm, vias 3 -> 0
- net VLED+: track 66.5 -> 0.00 mm, vias 4 -> 0
- net B2: track 64.6 -> 0.00 mm, vias 1 -> 0
- net ADV_Sync: track 64.5 -> 0.00 mm, vias 5 -> 0
- net B4: track 64.0 -> 0.00 mm, vias 1 -> 0
- net IO8_ATX: track 63.7 -> 0.00 mm
- net PCF_SDA: track 62.1 -> 0.03 mm, vias 3 -> 0
- net IO7_ATX: track 60.0 -> 0.00 mm
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Other:
- board text removed: "IO 3V3/5V"

Commit message: RGB
Connections:
- J5 pad 23: (no net) -> GND
- J5 pad 7: (no net) -> GND
- U1 pad 1: G7 -> G2
- U1 pad 2: B3 -> R7
- U1 pad 3: B4 -> R6
- U1 pad 4: B5 -> R5
- U1 pad 6: B6 -> R4
- U1 pad 7: B7 -> R3
- U1 pad 87: R3 -> B7
- U1 pad 89: R4 -> B6
- U1 pad 90: R5 -> B5
- U1 pad 91: R6 -> B4
- U1 pad 92: R7 -> B3
- U1 pad 93: G2 -> G7
- U1 pad 94: G3 -> G6
- U1 pad 95: G4 -> G5
- U1 pad 96: G5 -> G4
- U1 pad 97: G6 -> G3
Routing:
- net B4: track 0.00 -> 100.6 mm, vias 0 -> 1
- net B7: track 23.0 -> 113.5 mm
- net B6: track 24.5 -> 109.2 mm
- net B5: track 25.3 -> 105.0 mm
- net B3: track 20.0 -> 96.4 mm
- net G6: track 18.9 -> 87.2 mm, vias 0 -> 1
- net G7: track 25.3 -> 90.1 mm
- net (no net): track 74.2 -> 29.6 mm, vias 4 -> 2
- net G5: track 43.5 -> 84.3 mm, vias 0 -> 1
- net G4: track 45.8 -> 81.1 mm
- net R4: track 54.4 -> 85.9 mm
- net G3: track 46.6 -> 77.8 mm
- net R3: track 56.5 -> 82.1 mm
- net GND: track 1020.6 -> 1044.2 mm
- net R5: track 54.4 -> 77.7 mm
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