File: Sterownik CPLD dla TFT LCD.sch (KiCad schematic (older format))
At the start: 183 parts, among them J1 Conn_01x02, J10 5V select, J11 IO_5V, J13 VGA, J14 RGB_LSB, J15 Audio Out, J2 Conn_01x02, J3 PDI, J4 JTAG, J5 Conn_01x40, J6 Micro_SD_Card, J7 9V AC, J8 9V AC, J9 5V DC, Q1 BSS138, Q2 BSS138, Q3 BSS138, Q4 BSS138, Q5 BSS138, Q6 BSS138, Q7 BSS138, Q8 BSS138, SW1 Reset, SW2 IO_3V3_ON/OFF, U1 XC2C256_VQ100, U10 74LS573, U11 74AHC1G00, U12 LM1117-1.8, U13 L7805, U14 RT9293, U15 MIC2289_MILF8, U16 PCF8563T, U17 ADV7123_TQFP48, U18 TPA2005, U19 74AHCT1GU04, U2 LM1117-3.3, U20 74AHCT1GU04, U3 ATxmega128A1-AU, U4 NAND_Flash_TSOP48, U5 SRAM_1024Kx16bit_TSOP48I, U6 74AHC1G00, U7 SRAM_1024Kx16bit_TSOP48I, U8 74LS573, U9 SRAM_512Kx16bit_TSOP44II, X1 IQXO-70, X2 IQXO-70, Y1 32768Hz

Commit message: I-sze zmiany
Parts:
- removed C47, C48, C49, C50, C51, C52, C53, C54, C7: 100nF, Capacitor_SMD:C_1206_3216Metric, symbol Device:C
- removed C55: 2n2, Capacitor_SMD:C_1206_3216Metric, symbol Device:C
- removed D2: 1N5819, Diode_SMD:D_SOD-123, symbol Device:D
- removed D3: 1N4148, Diode_SMD:D_MiniMELF, symbol Device:D
- removed F1: Fuse, Fuse:Fuse_1812_4532Metric, symbol Device:Polyfuse_Small
- removed J1, J2: Conn_01x02, Jumper:SolderJumper-2_P1.3mm_Open_RoundedPad1.0x1.5mm, symbol Connector_Generic:Conn_01x02
- removed J10: 5V select, Connector_PinHeader_2.54mm:PinHeader_1x03_P2.54mm_Vertical, symbol Connector_Generic:Conn_01x03
- removed J11: IO_5V, Connector_PinHeader_2.54mm:PinHeader_2x11_P2.54mm_Horizontal, symbol Connector_Generic:Conn_02x11_Odd_Even
- removed J8: 9V AC, Jacek:Zlacze_srubowe_2x_5mm, symbol Connector_Generic:Conn_01x02
- removed L1: 10uH, Inductor_SMD:L_Taiyo-Yuden_NR-40xx, symbol Device:L
- removed L2: 22uH, Inductor_SMD:L_Taiyo-Yuden_NR-40xx, symbol Device:L
- removed Q3, Q4, Q5, Q6, Q7, Q8: BSS138, Package_TO_SOT_SMD:SOT-23, symbol Transistor_FET:BSS138
- removed R13: 2R2, Resistor_SMD:R_1206_3216Metric, symbol Device:R
- removed R14, R26, R27, R28, R29, R30, R31, R32, R33, R34, R35, R36, R37: 10k, Resistor_SMD:R_0603_1608Metric, symbol Device:R
- removed R15: 4k7, Resistor_SMD:R_1206_3216Metric, symbol Device:R
- removed R16: 7R5, Resistor_SMD:R_1206_3216Metric, symbol Device:R
- removed SW2: IO_3V3_ON/OFF, Button_Switch_THT:SW_DIP_SPSTx08_Slide_6.7x21.88mm_W7.62mm_P2.54mm_LowProfile, symbol Switch:SW_DIP_x08
- removed U14: RT9293, Package_TO_SOT_SMD:TSOT-23-6, symbol Jacek:RT9293
- removed U15: MIC2289_MILF8, Jacek:MLF8, symbol Jacek:MIC2289_MILF8
- removed X2: IQXO-70, Oscillator:Oscillator_SMD_IQD_IQXO70-4Pin_7.5x5.0mm, symbol Oscillator:IQXO-70
- U16: footprint Package_SO:SOIC-8_3.9x4.9mm_P1.27mm -> Package_SO:SO-8_3.9x4.9mm_P1.27mm
Connections:
- net 5V_DC is gone; now on net +5V: J9.1 (Pin_1)
- net IO4_ATX is gone; now on net SD_CD: U3.38 (PE3)
- net IO5_ATX is gone; now on net SD_CS: U3.39 (PE4)
- net IO6_ATX is gone; now on net SD_CLK: U3.40 (PE5)
- net IO7_ATX is gone; now on net SD_MISO: U3.41 (PE6)
- net IO8_ATX is gone; now on net SD_MOSI: U3.42 (PE7)
- net VLED+ is gone; now on net +5V: J5.2 (Pin_2)
- net VLED- is gone; now on net +5V: J5.1 (Pin_1)
- net +3V3: now also C6.1, X1.4 (V+)
- net ATX1: now also U1.16 (IO15), U3.11 (PB6); no longer U1.15 (IO14), U3.12 (PB7)
- net ATX10: now also U3.100 (PA5); no longer U3.96 (PA1)
- net ATX11: now also U3.99 (PA4); no longer U3.95 (AREF/PA0)
- net ATX12: now also U3.98 (PA3); no longer U3.88 (PQ3)
- net ATX13: now also U3.97 (PA2); no longer U3.87 (PQ2)
- net ATX14: now also U3.96 (PA1); no longer U3.86 (PQ1)
- net ATX15: now also U3.95 (AREF/PA0); no longer U3.85 (PQ0)
- net ATX2: now also U1.17 (IO16), U3.10 (PB5); no longer U1.16 (IO15), U3.11 (PB6)
- net ATX3: now also U1.18 (IO17), U3.9 (PB4); no longer U1.17 (IO16), U3.10 (PB5)
- net ATX4: now also U1.19 (IO18), U3.8 (PB3); no longer U1.18 (IO17), U3.9 (PB4)
- net ATX5: now also U1.22 (GCK0/IO19), U3.7 (PB2); no longer U1.19 (IO18), U3.8 (PB3)
- net ATX6: now also U3.6 (PB1); no longer U3.7 (PB2)
- net ATX7: now also U3.5 (AREF/PB0); no longer U3.6 (PB1)
- net ATX8: now also U3.2 (PA7); no longer U3.5 (AREF/PB0)
- net ATX9: now also U3.1 (PA6); no longer U3.97 (PA2)
- net B2: no longer U1.3 (GTS0/IO3), U17.18 (B4)
- net B3: now also U1.2 (GTS3/IO2); no longer U1.4 (GTS1/IO4)
- net B4: now also U1.3 (GTS0/IO3); no longer U1.6 (IO5)
- net B5: now also U1.4 (GTS1/IO4); no longer U1.7 (IO6)
- net B6: now also U1.6 (IO5); no longer U1.8 (IO7)
- net B7: now also U1.7 (IO6); no longer U1.9 (IO8)
- net CLK_Out: no longer U1.27 (GCK2/IO22)
- net DE: now also U1.12 (IO11); no longer U1.14 (IO13)
- net DISP: now also U1.9 (IO8); no longer U1.11 (IO10)
- net Ext_clk: now also U1.27 (GCK2/IO22); no longer U1.22 (GCK0/IO19)
- net G2: now also U1.93 (IO75); no longer U1.94 (IO76)
- net G3: now also U1.94 (IO76); no longer U1.95 (IO77)
- net G4: now also U1.95 (IO77); no longer U1.96 (IO78)
- net G5: now also U1.96 (IO78); no longer U1.97 (IO79)
- net G6: now also U1.97 (IO79); no longer U1.1 (GTS2/IO1)
- net G7: now also U1.1 (GTS2/IO1); no longer U1.2 (GTS3/IO2)
- net HSYNC: now also U1.10 (IO9); no longer U1.12 (IO11)
- net IO1_ATX: no longer U3.35 (PE0)
- net IO2_ATX: no longer U3.36 (PE1)
- net PCLK: now also U1.8 (IO7); no longer U1.10 (IO9)
- net R2: no longer U1.87 (IO70), U17.43 (R4)
- net R3: now also U1.87 (IO70); no longer U1.89 (IO71)
- net R4: now also U1.89 (IO71); no longer U1.90 (IO72)
- net R5: now also U1.90 (IO72); no longer U1.91 (IO73)
- net R6: now also U1.91 (IO73); no longer U1.92 (IO74)
- net R7: now also U1.92 (IO74); no longer U1.93 (IO75)
- net RGB_VCC_GND: now also U17.18 (B4), U17.43 (R4)
- net SD_CD: no longer U3.28 (PD3)
- net SD_CLK: no longer U3.30 (PD5)
- net SD_CS: no longer U3.29 (PD4)
- net SD_MISO: no longer U3.31 (PD6)
- net SD_MOSI: no longer U3.32 (PD7)
- net VSYNC: now also U1.11 (IO10); no longer U1.13 (IO12)
- net X+: no longer U3.99 (PA4)
- net X-: no longer U3.1 (PA6)
- net Y+: no longer U3.100 (PA5)
- net Y-: no longer U3.2 (PA7)
- net ATX_Clk: no longer names the net of U3.92 (PR1/XTAL1)
- net IO3_ATX: no longer names the net of U3.37 (PE2)
- net X1_EN: no longer names the net of X1.1 (E/B)
- net X1_EN: no longer U3.98 (PA3)
- net X2_EN: no longer names the net of U3.91 (PR0/XTAL2)
- new net ATX0: U1.15 (IO14), U3.12 (PB7)
Other:
- moved on the sheet: J9

Commit message: RGB
Connections:
- net B2 is gone; now on net GND: J5.23 (Pin_23)
- net R2 is gone; now on net GND: J5.7 (Pin_7)
- net B3: now also U1.92 (IO74); no longer U1.2 (GTS3/IO2)
- net B4: now also U1.91 (IO73); no longer U1.3 (GTS0/IO3)
- net B5: now also U1.90 (IO72); no longer U1.4 (GTS1/IO4)
- net B6: now also U1.89 (IO71); no longer U1.6 (IO5)
- net B7: now also U1.87 (IO70); no longer U1.7 (IO6)
- net G2: now also U1.1 (GTS2/IO1); no longer U1.93 (IO75)
- net G3: now also U1.97 (IO79); no longer U1.94 (IO76)
- net G4: now also U1.96 (IO78); no longer U1.95 (IO77)
- net G5: now also U1.95 (IO77); no longer U1.96 (IO78)
- net G6: now also U1.94 (IO76); no longer U1.97 (IO79)
- net G7: now also U1.93 (IO75); no longer U1.1 (GTS2/IO1)
- net R3: now also U1.7 (IO6); no longer U1.87 (IO70)
- net R4: now also U1.6 (IO5); no longer U1.89 (IO71)
- net R5: now also U1.4 (GTS1/IO4); no longer U1.90 (IO72)
- net R6: now also U1.3 (GTS0/IO3); no longer U1.91 (IO73)
- net R7: now also U1.2 (GTS3/IO2); no longer U1.92 (IO74)
Changed lines of the file:
@@
 Wire Wire Line
 	8750 5700 9275 5700
-Text GLabel 8750 2750 0    40   Input ~ 0
-R2
 Text GLabel 8750 2850 0    40   Input ~ 0
 R3
@@
 Text GLabel 8750 3250 0    40   Input ~ 0
 R7
-Text GLabel 8750 3550 0    40   Input ~ 0
-G2
 Text GLabel 8750 3650 0    40   Input ~ 0
 G3
@@
 Text GLabel 8750 4050 0    40   Input ~ 0
 G7
-Text GLabel 8750 4350 0    40   Input ~ 0
-B2
 Text GLabel 8750 4450 0    40   Input ~ 0
 B3
@@
 	1    0    0    -1
 $EndComp
-Wire Wire Line
-	8750 2650 8750 2700
-Wire Wire Line
-	8750 2700 9275 2700
-Connection ~ 8750 2650
 $Comp
 L power:GND #PWR026
@@
 	1    0    0    -1
 $EndComp
-Wire Wire Line
-	8750 3450 8750 3500
-Wire Wire Line
-	8750 3500 9275 3500
-Connection ~ 8750 3450
 $Comp
 L power:GND #PWR027
@@
 	1    0    0    -1
 $EndComp
-Wire Wire Line
-	8750 4250 8750 4300
-Wire Wire Line
-	8750 4300 9275 4300
-Connection ~ 8750 4250
-Text GLabel 4125 2925 2    40   Input ~ 0
+Text GLabel 2125 2425 0    40   Input ~ 0
 R3
-Text GLabel 4125 2825 2    40   Input ~ 0
+Text GLabel 2125 2325 0    40   Input ~ 0
 R4
-Text GLabel 4125 2725 2    40   Input ~ 0
+Text GLabel 2125 2225 0    40   Input ~ 0
 R5
-Text GLabel 4125 2625 2    40   Input ~ 0
+Text GLabel 2125 2125 0    40   Input ~ 0
 R6
-Text GLabel 4125 2525 2    40   Input ~ 0
+Text GLabel 2125 2025 0    40   Input ~ 0
 R7
-Text GLabel 4125 2425 2    40   Input ~ 0
+Text GLabel 2125 1925 0    40   Input ~ 0
 G2
-Text GLabel 4125 2325 2    40   Input ~ 0
+Text GLabel 4125 2025 2    40   Input ~ 0
 G3
-Text GLabel 4125 2225 2    40   Input ~ 0
-G4
 Text GLabel 4125 2125 2    40   Input ~ 0
+G4
+Text GLabel 4125 2225 2    40   Input ~ 0
 G5
-Text GLabel 4125 2025 2    40   Input ~ 0
+Text GLabel 4125 2325 2    40   Input ~ 0
 G6
-Text GLabel 2125 1925 0    40   Input ~ 0
+Text GLabel 4125 2425 2    40   Input ~ 0
 G7
-Text GLabel 2125 2025 0    40   Input ~ 0
+Text GLabel 4125 2525 2    40   Input ~ 0
 B3
-Text GLabel 2125 2125 0    40   Input ~ 0
+Text GLabel 4125 2625 2    40   Input ~ 0
 B4
-Text GLabel 2125 2225 0    40   Input ~ 0
+Text GLabel 4125 2725 2    40   Input ~ 0
 B5
-Text GLabel 2125 2325 0    40   Input ~ 0
+Text GLabel 4125 2825 2    40   Input ~ 0
 B6
-Text GLabel 2125 2425 0    40   Input ~ 0
+Text GLabel 4125 2925 2    40   Input ~ 0
 B7
 Text GLabel 2125 2525 0    40   Input ~ 0
@@
 	16375 11550 16375 11650
 Connection ~ 16375 11550
+Wire Wire Line
+	8750 2650 8750 2750
+Connection ~ 8750 2650
+Wire Wire Line
+	9275 2700 9275 2650
+Wire Wire Line
+	9275 2650 8750 2650
+Connection ~ 8750 3450
+Wire Wire Line
+	9275 3500 9275 3450
+Wire Wire Line
+	9275 3450 8750 3450
+Text GLabel 8750 3550 0    40   Input ~ 0
+G2
+Wire Wire Line
+	8750 4350 8750 4250
+Connection ~ 8750 4250
+Wire Wire Line
+	9275 4300 9275 4250
+Wire Wire Line
+	9275 4250 8750 4250
 $EndSCHEMATC
